Commit message: feat: add gazebo package

File: src2026_description/urdf/src2026.xacro (robot description, xacro)
@@ -444,6 +444,17 @@
     </collision>
   </link>
-  <link name="arm_3_virtual_link" />
-  <link name="shaft_virtual_link" />
+  <!-- Gazebo drops massless links while converting URDF to SDF.  Keep these
+       transmission links in the model with negligible inertia. -->
+  <xacro:macro name="virtual_link" params="name">
+    <link name="${name}">
+      <inertial>
+        <origin xyz="0 0 0" rpy="0 0 0" />
+        <mass value="0.001" />
+        <inertia ixx="1e-6" ixy="0" ixz="0" iyy="1e-6" iyz="0" izz="1e-6" />
+      </inertial>
+    </link>
+  </xacro:macro>
+  <xacro:virtual_link name="arm_3_virtual_link" />
+  <xacro:virtual_link name="shaft_virtual_link" />
   <link name="base_scan">
     <inertial>

Commit message: feat: QDD以外全部動いた

File: src2026_description/urdf/src2026.xacro (robot description, xacro)
@@ -6,5 +6,6 @@
   <xacro:arg name="can_interface" default="can0" />
   <xacro:arg name="drive_gear_ratio" default="19.0" />
-  <xacro:arg name="robomas_board_id" default="1" />
+  <xacro:arg name="robomas_board_id" default="3" />
+  <xacro:arg name="arm_y_module_id" default="6" />
   <xacro:arg name="servo_board_id" default="1" />
   <xacro:include filename="$(find src2026_description)/urdf/materials.xacro" />
@@ -545,5 +546,5 @@
     <axis xyz="-0.0 1.0 -0.0" />
   </joint>
-  <joint name="hand_right_joint" type="prismatic">
+  <joint name="gripper_joint" type="prismatic">
     <origin xyz="-0.1077 -7e-06 0.082" rpy="0 0 0" />
     <parent link="arm_4_link" />
@@ -557,5 +558,5 @@
     <child link="hand_left_link" />
     <axis xyz="1.0 0.0 0.0" />
-    <mimic joint="hand_right_joint" multiplier="1.0" offset="0.0" />
+    <mimic joint="gripper_joint" multiplier="1.0" offset="0.0" />
     <limit upper="0.07" lower="0.0" effort="100" velocity="100" />
   </joint>
@@ -564,4 +565,10 @@
     <parent link="base_link" />
     <child link="arm_1_link" />
+    <axis xyz="0.0 0.0 -1.0" />
+  </joint>
+  <link name="arm_y_link" />
+  <joint name="arm_y_joint" type="continuous">
+    <parent link="base_link" />
+    <child link="arm_y_link" />
     <axis xyz="0.0 0.0 -1.0" />
   </joint>

Commit message: feat: add odrive launcher

File: src2026_description/urdf/src2026.xacro (robot description, xacro)
@@ -4,4 +4,8 @@
   <xacro:arg name="use_fake_hardware" default="false" />
   <xacro:arg name="use_real_hardware" default="false" />
+  <xacro:arg name="enable_robot_hardware" default="true" />
+  <xacro:arg name="use_odrive_launcher" default="false" />
+  <xacro:arg name="odrive_can_interface" default="can1" />
+  <xacro:arg name="odrive_node_id" default="0" />
   <xacro:arg name="arm_only" default="false" />
   <xacro:arg name="drive_only" default="false" />
@@ -14,4 +18,11 @@
   <xacro:include filename="$(find src2026_description)/urdf/src2026.trans" />
   <xacro:include filename="$(find src2026_description)/urdf/src2026.gazebo" />
+  <link name="launcher_link"/>
+  <joint name="launcher_joint" type="continuous">
+    <origin xyz="0 0 0" rpy="0 0 0"/>
+    <parent link="base_link"/>
+    <child link="launcher_link"/>
+    <axis xyz="0 0 1"/>
+  </joint>
   <link name="base_footprint" />
   <joint name="base_link_joint" type="fixed">
